File: particle-somduino.kicad_pcb (KiCad board)
At the start: 2 copper layers, 68.6 x 53.3 mm, 30 parts, among them J1 1x08, J2 1x10, J3 1x06, J4 1x08, J5 Barrel_Jack_Switch, J6 Conn_01x02, J7 Conn_01x04, J8 USB_C_Receptacle_USB2.0_16P, SW1 SW_Push, SW2 SW_Push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

Commit message: tweaks
Connections:
- net Net-(D1-BK) renamed LED_B
- D1 pad 3: Net-(D1-GK) -> LED_R
- D1 pad 4: Net-(D1-RK) -> LED_G
- J8 pad A6: USB_D_N -> USB_D_P
- J8 pad A7: USB_D_P -> USB_D_N
- J8 pad B6: USB_D_N -> USB_D_P
- J8 pad B7: USB_D_P -> USB_D_N
- R1 pad 2: Net-(D1-RK) -> LED_R
- R2 pad 2: Net-(D1-GK) -> LED_G
Routing:
- net Net-(D1-RK): track 5.23 -> 0.00 mm
- net LED_G: track 0.00 -> 5.19 mm
- net Net-(D1-GK): track 3.48 -> 0.00 mm
- net LED_R: track 0.00 -> 3.07 mm
- net USB_D_P: track 28.0 -> 26.9 mm
- net USB_D_N: track 26.9 -> 27.8 mm
Other:
- board text added: "Somduino v2"
- board text removed: "Somduino v1"
