File: particle-somduino.kicad_sch (KiCad schematic)
At the start: 26 parts, among them J1 1x08, J2 1x10, J3 1x06, J4 1x08, J5 Barrel_Jack_Switch, J6 Conn_01x02, J7 Conn_01x04, J8 USB_C_Receptacle_USB2.0_16P, SW1 SW_Push, SW2 SW_Push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

Commit message: tweaks
Connections:
- net USB_D_N: now also J8.A7 (D-), J8.B7 (D-); no longer J8.A6 (D+), J8.B6 (D+)
- net USB_D_P: now also J8.A6 (D+), J8.B6 (D+); no longer J8.A7 (D-), J8.B7 (D-)
- net LED_B: now reaches D1.2 (BK), R3.2
- net LED_G: now reaches R2.2
- net LED_G: now also D1.4 (RK); no longer D1.3 (GK)
- net LED_R: now reaches R1.2
- net LED_R: now also D1.3 (GK); no longer D1.4 (RK)
Other:
- moved on the sheet: D1
Changed lines of the file:
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@@
 	(wire
 		(pts
+			(xy 265.43 158.75) (xy 267.97 158.75)
+		)
+		(stroke
+			(width 0)
+			(type default)
+		)
+	)
+	(wire
+		(pts
 			(xy 68.58 120.65) (xy 68.58 123.19)
 		)
@@
 	(wire
 		(pts
-			(xy 279.4 106.68) (xy 279.4 118.11)
+			(xy 281.94 142.24) (xy 281.94 153.67)
 		)
 		(stroke
@@
 	(wire
 		(pts
-			(xy 279.4 118.11) (xy 275.59 118.11)
+			(xy 281.94 153.67) (xy 278.13 153.67)
 		)
 		(stroke
@@
 	(wire
 		(pts
+			(xy 265.43 148.59) (xy 267.97 148.59)
+		)
+		(stroke
+			(width 0)
+			(type default)
+		)
+	)
+	(wire
+		(pts
 			(xy 62.23 120.65) (xy 68.58 120.65)
 		)
@@
 	(wire
 		(pts
+			(xy 265.43 153.67) (xy 267.97 153.67)
+		)
+		(stroke
+			(width 0)
+			(type default)
+		)
+	)
+	(wire
+		(pts
 			(xy 132.08 109.22) (xy 132.08 111.76)
 		)
@@
 	(global_label "USB_D_P"
 		(shape input)
-		(at 138.43 157.48 0)
+		(at 138.43 162.56 0)
 		(fields_autoplaced yes)
 		(effects
@@
 		)
 		(property "Intersheetrefs" "${INTERSHEET_REFS}"
-			(at 149.7955 157.48 0)
+			(at 149.7955 162.56 0)
 			(effects
 				(font
@@
 		)
 	)
+	(global_label "LED_B"
+		(shape input)
+		(at 265.43 158.75 180)
+		(fields_autoplaced yes)
+		(effects
+			(font
+				(size 1.27 1.27)
+			)
+			(justify right)
+		)
+		(property "Intersheetrefs" "${INTERSHEET_REFS}"
+			(at 256.665 158.75 0)
+			(effects
+				(font
+					(size 1.27 1.27)
+				)
+				(justify right)
+				(hide yes)
+			)
+		)
+	)
 	(global_label "A5"
 		(shape input)
@@
 		)
 	)
+	(global_label "LED_R"
+		(shape input)
+		(at 265.43 113.03 0)
+		(fields_autoplaced yes)
+		(effects
+			(font
+				(size 1.27 1.27)
+			)
+			(justify left)
+		)
+		(property "Intersheetrefs" "${INTERSHEET_REFS}"
+			(at 274.195 113.03 0)
+			(effects
+				(font
+					(size 1.27 1.27)
+				)
+				(justify left)
+				(hide yes)
+			)
+		)
+	)
 	(global_label "USB_D_N"
 		(shape input)
-		(at 138.43 162.56 0)
+		(at 138.43 157.48 0)
 		(fields_autoplaced yes)
 		(effects
@@
 		)
 		(property "Intersheetrefs" "${INTERSHEET_REFS}"
-			(at 149.856 162.56 0)
+			(at 149.856 157.48 0)
 			(effects
 				(font
@@
 		)
 	)
+	(global_label "LED_G"
+		(shape input)
+		(at 265.43 148.59 180)
+		(fields_autoplaced yes)
+		(effects
+			(font
+				(size 1.27 1.27)
+			)
+			(justify right)
+		)
+		(property "Intersheetrefs" "${INTERSHEET_REFS}"
+			(at 256.665 148.59 0)
+			(effects
+				(font
+					(size 1.27 1.27)
+				)
+				(justify right)
+				(hide yes)
+			)
+		)
+	)
+	(global_label "LED_G"
+		(shape input)
+		(at 265.43 118.11 0)
+		(fields_autoplaced yes)
+		(effects
+			(font
+				(size 1.27 1.27)
+			)
+			(justify left)
+		)
+		(property "Intersheetrefs" "${INTERSHEET_REFS}"
+			(at 274.195 118.11 0)
+			(effects
+				(font
+					(size 1.27 1.27)
+				)
+				(justify left)
+				(hide yes)
+			)
+		)
+	)
+	(global_label "LED_R"
+		(shape input)
+		(at 265.43 153.67 180)
+		(fields_autoplaced yes)
+		(effects
+			(font
+				(size 1.27 1.27)
+			)
+			(justify right)
+		)
+		(property "Intersheetrefs" "${INTERSHEET_REFS}"
+			(at 256.665 153.67 0)
+			(effects
+				(font
+					(size 1.27 1.27)
+				)
+				(justify right)
+				(hide yes)
+			)
+		)
+	)
 	(global_label "~{FUEL_INT}"
 		(shape input)
@@
 		)
 	)
+	(global_label "LED_B"
+		(shape input)
+		(at 265.43 123.19 0)
+		(fields_autoplaced yes)
+		(effects
+			(font
+				(size 1.27 1.27)
+			)
+			(justify left)
+		)
+		(property "Intersheetrefs" "${INTERSHEET_REFS}"
+			(at 274.195 123.19 0)
+			(effects
+				(font
+					(size 1.27 1.27)
+				)
+				(justify left)
+				(hide yes)
+			)
+		)
+	)
 	(global_label "D22"
 		(shape input)
@@
 	(symbol
 		(lib_id "Somduino_Symbols:LED_RGB")
-		(at 270.51 118.11 0)
+		(at 273.05 153.67 0)
 		(unit 1)
 		(exclude_from_sim no)
@@
 		(fields_autoplaced yes)
 		(property "Reference" "D1"
-			(at 270.51 104.14 0)
+			(at 273.05 139.7 0)
 			(effects
 				(font
@@
 		)
 		(property "Value" "LED_RGB"
-			(at 270.51 106.68 0)
+			(at 273.05 142.24 0)
 			(effects
 				(font
@@
 		)
 		(property "Footprint" "Somduino_Footprints:LED_RGB_Wuerth-PLCC4_3.2x2.8mm_150141M173100"
-			(at 270.51 105.41 0)
+			(at 273.05 140.97 0)
 			(effects
 				(font
@@
 		)
 		(property "Datasheet" ""
-			(at 270.51 129.54 0)
+			(at 273.05 165.1 0)
 			(effects
 				(font
@@
 		)
 		(property "Description" ""
-			(at 270.51 118.11 0)
+			(at 273.05 153.67 0)
 			(effects
 				(font
@@
 		)
 		(property "LCSC" "C5342281"
-			(at 270.51 118.11 0)
+			(at 273.05 153.67 0)
 			(effects
 				(font
@@
 	(symbol
 		(lib_id "power:+3V3")
-		(at 279.4 106.68 0)
+		(at 281.94 142.24 0)
 		(unit 1)
 		(exclude_from_sim no)
@@
 		(dnp no)
 		(property "Reference" "#PWR017"
-			(at 279.4 110.49 0)
+			(at 281.94 146.05 0)
 			(effects
 				(font
@@
 		)
 		(property "Value" "+3V3"
-			(at 279.4 101.6 90)
+			(at 281.94 137.16 90)
 			(effects
 				(font
@@
 		)
 		(property "Footprint" ""
-			(at 279.4 106.68 0)
+			(at 281.94 142.24 0)
 			(effects
 				(font
@@
 		)
 		(property "Datasheet" ""
-			(at 279.4 106.68 0)
+			(at 281.94 142.24 0)
 			(effects
 				(font
@@
 		)
 		(property "Description" "Power symbol creates a global label with name \"+3V3\""
-			(at 279.4 106.68 0)
+			(at 281.94 142.24 0)
 			(effects
 				(font
